File: kicad/AX5043.sch (KiCad schematic (older format))
At the start: 29 parts, among them U1 AX5043, X1 12.000MHz, X2 SMA

Commit message: Rescued some missing symbols/footprint in KiCad project
Parts:
- C1, C10, C11, C12, C13, C14, C15, C2, C3, C4, C5, C6, C7, C8, C9: symbol main-eagle-import:C-EUC0603 -> AX5043-rescue:C-EUC0603-main-eagle-import
- JP1: symbol main-eagle-import:PINHD-1X10 -> AX5043-rescue:PINHD-1X10-main-eagle-import
- R1, R10, R2, R3, R4, R5, R6, R7, R8, R9: symbol main-eagle-import:R-EU_R0603 -> AX5043-rescue:R-EU_R0603-main-eagle-import
- U1: symbol main-eagle-import:U-ONSEMI-AX5043 -> AX5043-rescue:U-ONSEMI-AX5043-main-eagle-import
- X1: symbol main-eagle-import:ASE -> AX5043-rescue:ASE-main-eagle-import
- X2: symbol main-eagle-import:SMA-142-0711-821_826 -> AX5043-rescue:SMA-142-0711-821_826-main-eagle-import
Changed lines of the file:
@@
 	3825 6200 3825 6300
 $Comp
-L main-eagle-import:U-ONSEMI-AX5043 U1
+L AX5043-rescue:U-ONSEMI-AX5043-main-eagle-import U1
 U 1 1 5C6255F6
 P 5625 4200
@@
 $EndComp
 $Comp
-L main-eagle-import:ASE X1
+L AX5043-rescue:ASE-main-eagle-import X1
 U 1 1 7C641B7C
 P 4125 1900
@@
 $EndComp
 $Comp
-L main-eagle-import:C-EUC0603 C1
+L AX5043-rescue:C-EUC0603-main-eagle-import C1
 U 1 1 C26272DC
 P 4825 1900
@@
 $EndComp
 $Comp
-L main-eagle-import:R-EU_R0603 R1
+L AX5043-rescue:R-EU_R0603-main-eagle-import R1
 U 1 1 BD41DF37
 P 3625 4700
@@
 $EndComp
 $Comp
-L main-eagle-import:C-EUC0603 C2
+L AX5043-rescue:C-EUC0603-main-eagle-import C2
 U 1 1 315DC9A5
 P 5125 2100
@@
 $EndComp
 $Comp
-L main-eagle-import:GND #GND01
+L AX5043-rescue:GND-main-eagle-import #GND01
 U 1 1 DB8695AC
 P 3525 2400
@@
 $EndComp
 $Comp
-L main-eagle-import:GND #GND02
+L AX5043-rescue:GND-main-eagle-import #GND02
 U 1 1 13A376EC
 P 4225 4000
@@
 $EndComp
 $Comp
-L main-eagle-import:GND #GND03
+L AX5043-rescue:GND-main-eagle-import #GND03
 U 1 1 7679BDCC
 P 4225 4600
@@
 $EndComp
 $Comp
-L main-eagle-import:GND #GND04
+L AX5043-rescue:GND-main-eagle-import #GND04
 U 1 1 D896219B
 P 5625 6400
@@
 $EndComp
 $Comp
-L main-eagle-import:R-EU_R0603 R2
+L AX5043-rescue:R-EU_R0603-main-eagle-import R2
 U 1 1 8547EDA2
 P 3625 3900
@@
 $EndComp
 $Comp
-L main-eagle-import:GND #GND05
+L AX5043-rescue:GND-main-eagle-import #GND05
 U 1 1 EF27308A
 P 3625 3500
@@
 $EndComp
 $Comp
-L main-eagle-import:GND #GND06
+L AX5043-rescue:GND-main-eagle-import #GND06
 U 1 1 A07C0193
 P 3625 5100
@@
 $EndComp
 $Comp
-L main-eagle-import:C-EUC0603 C3
+L AX5043-rescue:C-EUC0603-main-eagle-import C3
 U 1 1 36A1FDB1
 P 4725 3700
@@
 $EndComp
 $Comp
-L main-eagle-import:C-EUC0603 C4
+L AX5043-rescue:C-EUC0603-main-eagle-import C4
 U 1 1 14094E0B
 P 4725 4900
@@
 $EndComp
 $Comp
-L main-eagle-import:GND #GND07
+L AX5043-rescue:GND-main-eagle-import #GND07
 U 1 1 9CDE76EF
 P 5125 2400
@@
 $EndComp
 $Comp
-L main-eagle-import:SMA-142-0711-821_826 X2
+L AX5043-rescue:SMA-142-0711-821_826-main-eagle-import X2
 U 1 1 1303025E
 P 1325 4400
@@
 $EndComp
 $Comp
-L main-eagle-import:C-EUC0603 C5
+L AX5043-rescue:C-EUC0603-main-eagle-import C5
 U 1 1 F8E853AA
 P 3325 4200
@@
 $EndComp
 $Comp
-L main-eagle-import:C-EUC0603 C6
+L AX5043-rescue:C-EUC0603-main-eagle-import C6
 U 1 1 FF9C1704
 P 3325 4400
@@
 $EndComp
 $Comp
-L main-eagle-import:R-EU_R0603 R3
+L AX5043-rescue:R-EU_R0603-main-eagle-import R3
 U 1 1 516364D7
 P 2825 4200
@@
 $EndComp
 $Comp
-L main-eagle-import:R-EU_R0603 R4
+L AX5043-rescue:R-EU_R0603-main-eagle-import R4
 U 1 1 EFBD670E
 P 2825 4400
@@
 $EndComp
 $Comp
-L main-eagle-import:C-EUC0603 C7
+L AX5043-rescue:C-EUC0603-main-eagle-import C7
 U 1 1 4FD2610B
 P 2525 3900
@@
 $EndComp
 $Comp
-L main-eagle-import:R-EU_R0603 R5
+L AX5043-rescue:R-EU_R0603-main-eagle-import R5
 U 1 1 2E887318
 P 2225 4200
@@
 $EndComp
 $Comp
-L main-eagle-import:R-EU_R0603 R6
+L AX5043-rescue:R-EU_R0603-main-eagle-import R6
 U 1 1 BF0B7145
 P 2225 4700
@@
 $EndComp
 $Comp
-L main-eagle-import:C-EUC0603 C8
+L AX5043-rescue:C-EUC0603-main-eagle-import C8
 U 1 1 C72066DC
 P 2525 4700
@@
 $EndComp
 $Comp
-L main-eagle-import:GND #GND08
+L AX5043-rescue:GND-main-eagle-import #GND08
 U 1 1 DF24F9E8
 P 2525 3500
@@
 $EndComp
 $Comp
-L main-eagle-import:GND #GND09
+L AX5043-rescue:GND-main-eagle-import #GND09
 U 1 1 928DF91D
 P 2525 5100
@@
 $EndComp
 $Comp
-L main-eagle-import:GND #GND010
+L AX5043-rescue:GND-main-eagle-import #GND010
 U 1 1 845C69E3
 P 2225 5100
@@
 $EndComp
 $Comp
-L main-eagle-import:C-EUC0603 C9
+L AX5043-rescue:C-EUC0603-main-eagle-import C9
 U 1 1 0D7328F0
 P 1825 4400
@@
 $EndComp
 $Comp
-L main-eagle-import:GND #GND011
+L AX5043-rescue:GND-main-eagle-import #GND011
 U 1 1 19DA8D48
 P 1625 5100
@@
 $EndComp
 $Comp
-L main-eagle-import:R-EU_R0603 R7
+L AX5043-rescue:R-EU_R0603-main-eagle-import R7
 U 1 1 A7C90EEE
 P 3125 1200
@@
 $EndComp
 $Comp
-L main-eagle-import:C-EUC0603 C10
+L AX5043-rescue:C-EUC0603-main-eagle-import C10
 U 1 1 9CF4227D
 P 3825 1200
@@
 $EndComp
 $Comp
-L main-eagle-import:GND #GND012
+L AX5043-rescue:GND-main-eagle-import #GND012
 U 1 1 A5F18D96
 P 4025 1400
@@
 $EndComp
 $Comp
-L main-eagle-import:C-EUC0603 C11
+L AX5043-rescue:C-EUC0603-main-eagle-import C11
 U 1 1 59663956
 P 2825 1400
@@
 $EndComp
 $Comp
-L main-eagle-import:GND #GND013
+L AX5043-rescue:GND-main-eagle-import #GND013
 U 1 1 9E3D6951
 P 2825 1800
@@
 $EndComp
 $Comp
-L main-eagle-import:R-EU_R0603 R8
+L AX5043-rescue:R-EU_R0603-main-eagle-import R8
 U 1 1 8A1859B6
 P 5325 3200
@@
 $EndComp
 $Comp
-L main-eagle-import:C-EUC0603 C12
+L AX5043-rescue:C-EUC0603-main-eagle-import C12
 U 1 1 714954B3
 P 5925 3200
@@
 $EndComp
 $Comp
-L main-eagle-import:GND #GND014
+L AX5043-rescue:GND-main-eagle-import #GND014
 U 1 1 109F320A
 P 6225 3400
@@
 $EndComp
 $Comp
-L main-eagle-import:+3V3 #+3V01
+L AX5043-rescue:+3V3-main-eagle-import #+3V01
 U 1 1 406B5002
 P 5025 3000
@@
 $EndComp
 $Comp
-L main-eagle-import:+3V3 #+3V02
+L AX5043-rescue:+3V3-main-eagle-import #+3V02
 U 1 1 37D36547
 P 2825 1000
@@
 $EndComp
 $Comp
-L main-eagle-import:C-EUC0603 C13
+L AX5043-rescue:C-EUC0603-main-eagle-import C13
 U 1 1 9AFB8C1C
 P 4725 3200
@@
 $EndComp
 $Comp
-L main-eagle-import:GND #GND015
+L AX5043-rescue:GND-main-eagle-import #GND015
 U 1 1 257B06B4
 P 4225 3200
@@
 $EndComp
 $Comp
-L main-eagle-import:R-EU_R0603 R9
+L AX5043-rescue:R-EU_R0603-main-eagle-import R9
 U 1 1 4584D8AF
 P 4625 5800
@@
 $EndComp
 $Comp
-L main-eagle-import:C-EUC0603 C14
+L AX5043-rescue:C-EUC0603-main-eagle-import C14
 U 1 1 4270E9F2
 P 4125 6200
@@
 $EndComp
 $Comp
-L main-eagle-import:R-EU_R0603 R10
+L AX5043-rescue:R-EU_R0603-main-eagle-import R10
 U 1 1 4E9AE05B
 P 3825 6000
@@
 $EndComp
 $Comp
-L main-eagle-import:C-EUC0603 C15
+L AX5043-rescue:C-EUC0603-main-eagle-import C15
 U 1 1 BE83EA0E
 P 3825 6400
@@
 $EndComp
 $Comp
-L main-eagle-import:GND #GND016
+L AX5043-rescue:GND-main-eagle-import #GND016
 U 1 1 99D4D269
 P 3825 6900
@@
 $EndComp
 $Comp
-L main-eagle-import:GND #GND017
+L AX5043-rescue:GND-main-eagle-import #GND017
 U 1 1 0A5A0AC8
 P 4125 6900
@@
 $EndComp
 $Comp
-L main-eagle-import:DINA4_L #FRAME1
+L AX5043-rescue:DINA4_L-main-eagle-import #FRAME1
 U 1 1 73DA64CA
 P 900 7400
@@
 $EndComp
 $Comp
-L main-eagle-import:PINHD-1X10 JP1
+L AX5043-rescue:PINHD-1X10-main-eagle-import JP1
 U 1 1 2F430EF2
 P 9825 3300
@@
 $EndComp
 $Comp
-L main-eagle-import:GND #GND018
+L AX5043-rescue:GND-main-eagle-import #GND018
 U 1 1 E0081D19
 P 9425 4100
@@
 $EndComp
 $Comp
-L main-eagle-import:+3V3 #+3V03
+L AX5043-rescue:+3V3-main-eagle-import #+3V03
 U 1 1 A56F219E
 P 9425 2600

Commit message: Reorganised KiCad libraries
Parts:
- C1, C10, C11, C12, C13, C14, C15, C2, C3, C4, C5, C6, C7, C8, C9: footprint main:C0603 -> AX5043:C0603; symbol AX5043-rescue:C-EUC0603-main-eagle-import -> AX5043:C-EUC0603
- JP1: footprint main:1X10 -> AX5043:1X10; symbol AX5043-rescue:PINHD-1X10-main-eagle-import -> AX5043:PINHD-1X10
- R1, R10, R2, R3, R4, R5, R6, R7, R8, R9: footprint main:R0603 -> AX5043:R0603; symbol AX5043-rescue:R-EU_R0603-main-eagle-import -> AX5043:R-EU_R0603
- U1: footprint main:QFN28-5X5-WITH-CENTER-PAD -> AX5043:QFN28-5X5-WITH-CENTER-PAD; symbol AX5043-rescue:U-ONSEMI-AX5043-main-eagle-import -> AX5043:U-ONSEMI-AX5043
- X1: footprint main:ASE -> AX5043:ASE; symbol AX5043-rescue:ASE-main-eagle-import -> AX5043:ASE
- X2: footprint main:J502-ND-142-0711-821_826 -> AX5043:J502-ND-142-0711-821_826; symbol AX5043-rescue:SMA-142-0711-821_826-main-eagle-import -> AX5043:SMA-142-0711-821_826

Commit message: New footprint for TCXO, model is ECS-TXO-2520
Parts:
- X1: footprint AX5043:ASE -> AX5043:ECS-TXO-2520
Changed lines of the file:
@@
 F 0 "X1" H 3825 2225 59  0000 L BNN
 F 1 "12.000MHz" H 3825 1500 59  0000 L BNN
-F 2 "AX5043:ASE" H 4125 1900 50  0001 C CNN
+F 2 "AX5043:ECS-TXO-2520" H 4125 1900 50  0001 C CNN
 F 3 "" H 4125 1900 50  0001 C CNN
 	1    4125 1900
